Commit message: Project Map my world added

File: src/my_robot/urdf/my_robot.xacro (robot description, xacro)
@@ -186,4 +186,11 @@
        <axis xyz="0 1 0" rpy="0 0 0"/>
     </joint>
+   <joint name="camera_optical_joint" type="fixed">
+    <origin xyz="0 0 0" rpy="-1.5707 0 -1.5707"/>
+    <parent link="camera"/>
+    <child link="camera_link_optical"/>
+  </joint>
+  <link name="camera_link_optical">
+  </link>
    <link name="hokuyo">
       <inertial>
